File: bitraf-rpi-breakout.brd (EAGLE design)
At the start: 65.7 x 57.1 mm, 20 parts, among them IC1 74HC595N, K1 JS-M1-9V-4, T1 BC547

Commit message: Rev b.
Parts:
- D1, D2: value (none) -> 3.3V
- D3: value 1N4148DO35-7 -> 1N4004; device diode:DO35-7 -> diode:DO41-10
- R1, R2, R3, R4: value (none) -> 330
- R6, R7: value (none) -> 4.7k
- moved SV1 6.99 mm to (4.76, 29.8), turned to 90 degrees
- moved LED1 6.70 mm to (53.0, 40.0)
- moved R1 5.79 mm to (39.1, 40.0)
- moved LED2 5.65 mm to (53.0, 46.4)
- moved R5 5.17 mm to (30.2, 24.1)
- moved LED3 4.55 mm to (50.5, 34.9)
- moved R2 4.55 mm to (39.1, 46.4)
- moved R4 4.55 mm to (39.1, 34.9)
- moved IC1 4.55 mm to (21.3, 37.5)
- moved R6 3.31 mm to (54.3, 26.0)
- moved R7 3.31 mm to (54.3, 28.6)
- moved JP1 3.19 mm to (62.5, 27.3)
- moved D2 2.93 mm to (42.9, 22.2)
- moved D1 2.31 mm to (46.7, 24.8)
- moved LED4 2.13 mm to (50.5, 32.4)
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Routing:
- net VCC: track 115.6 -> 162.0 mm, vias 4 -> 0
- net N$20: track 31.6 -> 12.0 mm
- net N$8: track 45.8 -> 64.8 mm
- net N$9: track 45.8 -> 56.2 mm
- net GND: track 211.2 -> 203.4 mm
- net N$19: track 13.8 -> 19.2 mm
- net N$21: track 17.9 -> 13.0 mm
- net N$6: track 27.3 -> 24.4 mm
- net N$2: track 6.35 -> 8.89 mm
- net N$1: track 6.35 -> 8.89 mm
- net N$12: track 15.3 -> 14.1 mm
- net TTL_IN_2: track 3.81 -> 3.18 mm
- net TTL_IN_1: track 3.81 -> 3.18 mm
- net N$5: track 10.2 -> 10.7 mm
Other:
- board size 65.7 x 57.1 mm -> 66.7 x 48.9 mm
- board text added: "Bitraf R-π Brk 2013 Rev B"

Commit message: nits
Parts:
- moved T1 12.6 mm to (23.8, 14.6)
Connections:
- net GND: no longer IC1.10
- net VCC: now also IC1.10
Routing:
- net VCC: track 162.0 -> 190.2 mm
- net N$15: track 32.7 -> 14.0 mm
- net N$6: track 24.4 -> 12.3 mm
- net GND: track 203.4 -> 199.7 mm

Commit message: o Changing relay.
Parts:
- J1: device con-amp:1X3MTA -> con-amp:1X2MTA
- K1: value JS-M1-9V-4 -> FTR-F3FTR-F3AA005E; device relay:JS-M -> fujitsu-ftr-f3:REED
- moved K1 11.5 mm to (34.9, 4.76), turned to 0 degrees
Connections:
- removed net N$18: J1.3, K1.NC
- net N$15: now also K1.4; no longer K1.2
- net N$16: now also K1.2; no longer K1.C
- net N$17: now also K1.1; no longer K1.NO
- net VCC: now also K1.3; no longer K1.1
Routing:
- net N$16: track 25.2 -> 7.91 mm
- net N$18: track 11.8 -> 0.00 mm
- net VCC: track 190.2 -> 184.6 mm
- net N$17: track 11.9 -> 15.1 mm
- net N$15: track 14.0 -> 15.4 mm
Changed lines of the file:
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@@
 <param name="mdSmdStop" value="0mil"/>
 <param name="msWidth" value="10mil"/>
-<param name="msDrill" value="24mil"/>
+<param name="msDrill" value="0.4mm"/>
 <param name="msMicroVia" value="9.99mm"/>
 <param name="msBlindViaRatio" value="0.5"/>
@@
 <element name="IC1" library="74xx-eu" package="DIL16" value="74HC595N" x="21.2725" y="37.465" rot="R90"/>
 <element name="T1" library="transistor" package="TO92" value="BC547" x="23.8125" y="14.605" rot="R180"/>
-<element name="K1" library="relay" package="JS-M" value="JS-M1-9V-4" x="45.4025" y="9.525" rot="R180">
-<attribute name="OC_NEWARK" value="unknown" x="21.2725" y="18.415" size="1.778" layer="27" rot="R180" display="off"/>
-<attribute name="MPN" value="" x="21.2725" y="18.415" size="1.778" layer="27" rot="R180" display="off"/>
-<attribute name="MF" value="" x="21.2725" y="18.415" size="1.778" layer="27" rot="R180" display="off"/>
-<attribute name="OC_FARNELL" value="unknown" x="21.2725" y="18.415" size="1.778" layer="27" rot="R180" display="off"/>
-</element>
 <element name="R1" library="resistor" package="0204/7" value="330" x="39.0525" y="40.005"/>
 <element name="R2" library="resistor" package="0204/7" value="330" x="39.0525" y="46.355"/>
@@
 </element>
 <element name="JP1" library="pinhead" package="2X02" value="" x="62.5475" y="27.305"/>
-<element name="J1" library="con-amp" package="1X3MTA" value="" x="61.9125" y="9.525" rot="R270"/>
+<element name="J1" library="con-amp" package="1X2MTA" value="" x="61.9125" y="9.525" rot="R270"/>
+<element name="K1" library="fujitsu-ftr-f3" package="REED" value="FTR-F3FTR-F3AA005E" x="34.925" y="4.7625">
+<attribute name="OC_NEWARK" value="" x="34.925" y="4.7625" size="1.778" layer="27" display="off"/>
+<attribute name="MPN" value="" x="34.925" y="4.7625" size="1.778" layer="27" display="off"/>
+<attribute name="MF" value="" x="34.925" y="4.7625" size="1.778" layer="27" display="off"/>
+<attribute name="MOUSER" value="817-FTR-F3AA005E" x="34.925" y="4.7625" size="1.778" layer="27" display="off"/>
+<attribute name="OC_FARNELL" value="" x="34.925" y="4.7625" size="1.778" layer="27" display="off"/>
+</element>
 </elements>
 <signals>
@@
 <signal name="VCC">
 <contactref element="IC1" pad="16"/>
-<contactref element="K1" pad="1"/>
 <contactref element="D3" pad="C"/>
 <contactref element="SV1" pad="2"/>
 <contactref element="JP1" pad="4"/>
-<wire x1="59.3725" y1="18.415" x2="46.6725" y2="18.415" width="0.4064" layer="16"/>
-<wire x1="46.6725" y1="18.415" x2="40.3225" y2="12.065" width="0.4064" layer="16"/>
-<wire x1="40.3225" y1="12.065" x2="36.5125" y2="12.065" width="0.4064" layer="16"/>
-<wire x1="36.5125" y1="12.065" x2="34.6075" y2="10.16" width="0.4064" layer="16"/>
-<wire x1="34.6075" y1="10.16" x2="34.6075" y2="4.445" width="0.4064" layer="16"/>
+<wire x1="59.3725" y1="18.415" x2="45.4025" y2="18.415" width="0.4064" layer="16"/>
 <wire x1="62.5475" y1="22.225" x2="59.3725" y2="18.415" width="0.4064" layer="16"/>
 <wire x1="63.8175" y1="28.575" x2="62.5475" y2="27.305" width="0.4064" layer="16"/>
@@
 <wire x1="51.1175" y1="24.13" x2="41.5925" y2="24.13" width="0.4064" layer="16"/>
 <wire x1="41.5925" y1="24.13" x2="40.3225" y2="22.86" width="0.4064" layer="16"/>
-<wire x1="40.3225" y1="22.86" x2="16.8275" y2="22.86" width="0.4064" layer="16"/>
-<wire x1="40.3225" y1="22.86" x2="40.3225" y2="12.065" width="0.4064" layer="16"/>
-<wire x1="28.8925" y1="4.445" x2="34.6075" y2="4.445" width="0.4064" layer="16"/>
-<wire x1="34.6075" y1="4.445" x2="37.7825" y2="4.445" width="0.4064" layer="16"/>
-<wire x1="37.7825" y1="4.445" x2="38.7025" y2="3.525" width="0.4064" layer="16"/>
+<wire x1="40.3225" y1="22.86" x2="38.735" y2="22.86" width="0.4064" layer="16"/>
+<wire x1="38.735" y1="22.86" x2="16.8275" y2="22.86" width="0.4064" layer="16"/>
+<wire x1="28.8925" y1="4.445" x2="37.7825" y2="4.445" width="0.4064" layer="16"/>
 <contactref element="IC1" pad="10"/>
 <wire x1="17.4625" y1="43.815" x2="18.415" y2="43.815" width="0.4064" layer="16"/>
@@
 <wire x1="4.445" y1="12.065" x2="6.0325" y2="12.065" width="0.4064" layer="16"/>
 <wire x1="6.0325" y1="12.065" x2="16.8275" y2="22.86" width="0.4064" layer="16"/>
+<contactref element="K1" pad="3"/>
+<wire x1="38.945" y1="6.0125" x2="38.945" y2="5.6075" width="0.4064" layer="16"/>
+<wire x1="38.945" y1="5.6075" x2="37.7825" y2="4.445" width="0.4064" layer="16"/>
+<wire x1="38.945" y1="6.0125" x2="38.945" y2="16.1925" width="0.4064" layer="16"/>
+<wire x1="38.945" y1="16.1925" x2="38.945" y2="22.65" width="0.4064" layer="16"/>
+<wire x1="38.945" y1="22.65" x2="38.735" y2="22.86" width="0.4064" layer="16"/>
+<wire x1="45.4025" y1="18.415" x2="43.18" y2="16.1925" width="0.4064" layer="16"/>
+<wire x1="43.18" y1="16.1925" x2="38.945" y2="16.1925" width="0.4064" layer="16"/>
 </signal>
 <signal name="N$1">
@@
 </signal>
 <signal name="N$15">
-<contactref element="K1" pad="2"/>
 <contactref element="T1" pad="3"/>
 <contactref element="D3" pad="A"/>
+<contactref element="K1" pad="4"/>
 <wire x1="25.0825" y1="14.605" x2="28.8925" y2="14.605" width="0.4064" layer="16"/>
-<wire x1="28.8925" y1="14.605" x2="37.7825" y2="14.605" width="0.4064" layer="16"/>
-<wire x1="37.7825" y1="14.605" x2="38.7025" y2="15.525" width="0.4064" layer="16"/>
-</signal>
-<signal name="N$16" class="1">
-<contactref element="K1" pad="C"/>
-<contactref element="J1" pad="2"/>
-<wire x1="36.7279" y1="9.5504" x2="61.9125" y2="9.5504" width="1.778" layer="16"/>
-<wire x1="36.7279" y1="9.5504" x2="36.7025" y2="9.525" width="1.778" layer="16"/>
-</signal>
-<signal name="N$17" class="1">
-<contactref element="K1" pad="NO"/>
-<contactref element="J1" pad="1"/>
-<wire x1="50.9025" y1="3.525" x2="59.8495" y2="3.525" width="1.778" layer="16"/>
-<wire x1="59.8495" y1="3.525" x2="61.9125" y2="5.588" width="1.778" layer="16"/>
-</signal>
-<signal name="N$18" class="1">
-<contactref element="K1" pad="NC"/>
-<contactref element="J1" pad="3"/>
-<wire x1="50.9025" y1="15.525" x2="59.9003" y2="15.525" width="1.778" layer="16"/>
-<wire x1="59.9003" y1="15.525" x2="61.9125" y2="13.5128" width="1.778" layer="16"/>
+<wire x1="28.8925" y1="14.605" x2="36.195" y2="7.3025" width="0.4064" layer="16"/>
+<wire x1="36.195" y1="7.3025" x2="36.195" y2="6.0625" width="0.4064" layer="16"/>
+<wire x1="36.195" y1="6.0625" x2="36.245" y2="6.0125" width="0.4064" layer="16"/>
 </signal>
 <signal name="N$20">
@@
 </polygon>
 </signal>
+<signal name="N$16" class="1">
+<contactref element="K1" pad="2"/>
+<contactref element="J1" pad="2"/>
+<wire x1="61.9125" y1="11.5062" x2="56.5387" y2="11.5062" width="1.778" layer="16"/>
+<wire x1="56.5387" y1="11.5062" x2="54.745" y2="9.7125" width="1.778" layer="16"/>
+</signal>
+<signal name="N$17" class="1">
+<contactref element="J1" pad="1"/>
+<contactref element="K1" pad="1"/>
+<wire x1="61.9125" y1="7.5438" x2="49.9137" y2="7.5438" width="1.778" layer="16"/>
+<wire x1="49.9137" y1="7.5438" x2="47.745" y2="9.7125" width="1.778" layer="16"/>
+</signal>
 </signals>

Commit message: o Relay was upside down.
Parts:
- moved K1 0.63 mm to (34.9, 5.40)
Connections:
- net N$16: now also J1.1; no longer J1.2
- net N$17: now also J1.2; no longer J1.1
Routing:
- net N$15: track 15.4 -> 14.2 mm
- net N$17: track 15.1 -> 15.8 mm
- net N$16: track 7.91 -> 7.21 mm
Changed lines of the file:
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@@
 <setting verticaltext="up"/>
 </settings>
-<grid distance="0.0125" unitdist="inch" unit="inch" style="lines" multiple="1" display="no" altdistance="0.1" altunitdist="mm" altunit="mm"/>
+<grid distance="25" unitdist="mil" unit="mil" style="lines" multiple="1" display="no" altdistance="0.1" altunitdist="mm" altunit="mm"/>
 <layers>
 <layer number="1" name="Top" color="4" fill="1" visible="yes" active="yes"/>
@@
 <element name="JP1" library="pinhead" package="2X02" value="" x="62.5475" y="27.305"/>
 <element name="J1" library="con-amp" package="1X2MTA" value="" x="61.9125" y="9.525" rot="R270"/>
-<element name="K1" library="fujitsu-ftr-f3" package="REED" value="FTR-F3FTR-F3AA005E" x="34.925" y="4.7625">
-<attribute name="OC_NEWARK" value="" x="34.925" y="4.7625" size="1.778" layer="27" display="off"/>
-<attribute name="MPN" value="" x="34.925" y="4.7625" size="1.778" layer="27" display="off"/>
-<attribute name="MF" value="" x="34.925" y="4.7625" size="1.778" layer="27" display="off"/>
-<attribute name="MOUSER" value="817-FTR-F3AA005E" x="34.925" y="4.7625" size="1.778" layer="27" display="off"/>
-<attribute name="OC_FARNELL" value="" x="34.925" y="4.7625" size="1.778" layer="27" display="off"/>
+<element name="K1" library="fujitsu-ftr-f3" package="REED" value="FTR-F3FTR-F3AA005E" x="34.925" y="5.3975">
+<attribute name="OC_NEWARK" value="" x="34.925" y="5.3975" size="1.778" layer="27" display="off"/>
+<attribute name="MPN" value="" x="34.925" y="5.3975" size="1.778" layer="27" display="off"/>
+<attribute name="MF" value="" x="34.925" y="5.3975" size="1.778" layer="27" display="off"/>
+<attribute name="MOUSER" value="817-FTR-F3AA005E" x="34.925" y="5.3975" size="1.778" layer="27" display="off"/>
+<attribute name="OC_FARNELL" value="" x="34.925" y="5.3975" size="1.778" layer="27" display="off"/>
 </element>
 </elements>
@@
 <wire x1="6.0325" y1="12.065" x2="16.8275" y2="22.86" width="0.4064" layer="16"/>
 <contactref element="K1" pad="3"/>
-<wire x1="38.945" y1="6.0125" x2="38.945" y2="5.6075" width="0.4064" layer="16"/>
 <wire x1="38.945" y1="5.6075" x2="37.7825" y2="4.445" width="0.4064" layer="16"/>
-<wire x1="38.945" y1="6.0125" x2="38.945" y2="16.1925" width="0.4064" layer="16"/>
 <wire x1="38.945" y1="16.1925" x2="38.945" y2="22.65" width="0.4064" layer="16"/>
 <wire x1="38.945" y1="22.65" x2="38.735" y2="22.86" width="0.4064" layer="16"/>
 <wire x1="45.4025" y1="18.415" x2="43.18" y2="16.1925" width="0.4064" layer="16"/>
 <wire x1="43.18" y1="16.1925" x2="38.945" y2="16.1925" width="0.4064" layer="16"/>
+<wire x1="38.945" y1="5.6075" x2="38.945" y2="11.1475" width="0.4064" layer="16"/>
+<wire x1="38.945" y1="16.1925" x2="38.945" y2="11.1475" width="0.4064" layer="16"/>
 </signal>
 <signal name="N$1">
@@
 <contactref element="K1" pad="4"/>
 <wire x1="25.0825" y1="14.605" x2="28.8925" y2="14.605" width="0.4064" layer="16"/>
-<wire x1="28.8925" y1="14.605" x2="36.195" y2="7.3025" width="0.4064" layer="16"/>
-<wire x1="36.195" y1="7.3025" x2="36.195" y2="6.0625" width="0.4064" layer="16"/>
-<wire x1="36.195" y1="6.0625" x2="36.245" y2="6.0125" width="0.4064" layer="16"/>
+<wire x1="28.8925" y1="14.605" x2="35.56" y2="14.605" width="0.4064" layer="16"/>
+<wire x1="35.56" y1="14.605" x2="36.195" y2="13.97" width="0.4064" layer="16"/>
+<wire x1="36.195" y1="13.97" x2="36.195" y2="11.1975" width="0.4064" layer="16"/>
+<wire x1="36.195" y1="11.1975" x2="36.245" y2="11.1475" width="0.4064" layer="16"/>
 </signal>
 <signal name="N$20">
@@
 <signal name="N$16" class="1">
 <contactref element="K1" pad="2"/>
+<contactref element="J1" pad="1"/>
+<wire x1="61.9125" y1="7.5438" x2="54.8413" y2="7.5438" width="1.9304" layer="16"/>
+<wire x1="54.8413" y1="7.5438" x2="54.745" y2="7.4475" width="0.4064" layer="16"/>
+</signal>
+<signal name="N$17" class="1">
+<contactref element="K1" pad="1"/>
 <contactref element="J1" pad="2"/>
-<wire x1="61.9125" y1="11.5062" x2="56.5387" y2="11.5062" width="1.778" layer="16"/>
-<wire x1="56.5387" y1="11.5062" x2="54.745" y2="9.7125" width="1.778" layer="16"/>
-</signal>
-<signal name="N$17" class="1">
-<contactref element="J1" pad="1"/>
-<contactref element="K1" pad="1"/>
-<wire x1="61.9125" y1="7.5438" x2="49.9137" y2="7.5438" width="1.778" layer="16"/>
-<wire x1="49.9137" y1="7.5438" x2="47.745" y2="9.7125" width="1.778" layer="16"/>
+<wire x1="61.9125" y1="11.5062" x2="51.8037" y2="11.5062" width="1.9304" layer="16"/>
+<wire x1="51.8037" y1="11.5062" x2="47.745" y2="7.4475" width="1.9304" layer="16"/>
 </signal>
 </signals>
